File: PCBs/MainBoard/Kicad_MiniSumo.kicad_pcb (KiCad board)
At the start: 2 copper layers, 92 x 32 mm, 18 parts, among them J1 Screw_Terminal_01x15, M2 MountingHole_2.2mm_M2

Commit message: Added information on PCB to change pads to thermal releases in next version!
Other:
- board text added: "CHANGE PADS TO THERMAL RELEASES IN NEXT VERSION!!!"
Changed lines of the file:
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@@
+		)
+	)
+	(gr_text "CHANGE PADS TO THERMAL RELEASES IN NEXT VERSION!!!"
+		(at 130.556 62.103 0)
+		(layer "F.Fab")
+		(effects
+			(font
+				(size 1.5 1.5)
+				(thickness 0.3)
+				(bold yes)
+			)
+			(justify left bottom)
 		)
 	)

Commit message: Project: add information about CN16 jumper to the PCB project
Other:
- board text added: "REMOVE CN16 ON NUCLEO BOARD BEFORE SOLDIERING"
Changed lines of the file:
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@@
+		)
+	)
+	(gr_text "REMOVE CN16 ON NUCLEO BOARD BEFORE SOLDIERING"
+		(at 131.572 59.055 0)
+		(layer "F.Fab")
+		(effects
+			(font
+				(size 1.5 1.5)
+				(thickness 0.3)
+				(bold yes)
+			)
+			(justify left bottom)
 		)
 	)

Commit message: Project: add new comment about THTs on the main PCB board
Other:
- board text added: "MAKE BIGGER THTs (to the size of STM one)"
Changed lines of the file:
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@@
+		)
+	)
+	(gr_text "MAKE BIGGER THTs (to the size of STM one)"
+		(at 136.398 55.753 0)
+		(layer "F.Fab")
+		(effects
+			(font
+				(size 1.5 1.5)
+				(thickness 0.3)
+				(bold yes)
+			)
+			(justify left bottom)
 		)
 	)
